Commit message: URDF fix

File: files_to_change/spot.urdf.xacro (robot description, xacro)
@@ -5,6 +5,4 @@
   <!-- Macros for loading the ROS 2 control tags -->
   <xacro:include filename="$(find spot_description)/urdf/spot.ros2_control.xacro" />
-  <!-- Include Velodyne VLP-16 URDF macro -->
-  <xacro:include filename="$(find velodyne_description)/urdf/VLP-16.urdf.xacro"/>
   <!-- General parameters -->
   <!-- String that will be prepended to all joints and links-->
@@ -49,13 +47,3 @@
                                k_qd_p="$(arg k_qd_p)" />
   </xacro:if>
-  <!-- Add Velodyne sensor to Spot -->
-  <!-- Instantiate the Velodyne macro -->
-  <xacro:vlp_16 name="velodyne_top"/>
-  <!-- Fixed joint to mount Velodyne on Spot's body -->
-  <joint name="velodyne_mount_joint" type="fixed">
-    <parent link="body"/> <!-- Replace 'body' with the main top frame of Spot if different -->
-    <child link="velodyne_top_base_link"/>
-    <!-- Position above the robot: 0.25m above, no rotation -->
-    <origin xyz="-0.183 0 0.1518" rpy="0 0 0"/>
-  </joint>
 </robot>

File: files_to_change/spot_macro.xacro (robot description, xacro)
@@ -402,13 +402,9 @@
             <limit effort="115" velocity="12.0" lower="-2.7929" upper="-0.257725" />
         </joint>
-        <!-- Add Velodyne -->
-        <xacro:vlp_16 name="velodyne_top"/>
-        <!-- Fixed joint to mount Velodyne on Spot's body -->
-        <joint name="${tf_prefix}velodyne_mount_joint" type="fixed">
-            <parent link="${tf_prefix}body"/> <!-- Replace 'body' with the main top frame of Spot if different -->
-            <child link="velodyne_top_base_link"/>
-            <!-- Position above the robot -->
+        <!-- Velodyne VLP-16 -->
+        <xacro:VLP-16 name="${tf_prefix}vlp16" parent="${tf_prefix}body">
+            <!-- adjust pose as needed -->
             <origin xyz="-0.183 0 0.1518" rpy="0 0 0"/>
-        </joint>
+        </xacro:VLP-16>
         <!-- Standard accessories. -->
         <xacro:include filename="$(find spot_description)/urdf/accessories.urdf.xacro" />
